File: 2026-tractor.kicad_sch (KiCad schematic)
At the start: 1 part, among them U1 4060

Commit message: Test commit
Parts:
- removed U1: 4060, symbol 4xxx:4060
Changed lines of the file:
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@@
 	(generator_version "9.0")
 	(paper "A4")
-	(symbol
-		(lib_id "4xxx:4060")
-		(at 95.25 73.66 0)
-		(unit 1)
-		(exclude_from_sim no)
-		(in_bom yes)
-		(on_board yes)
-		(dnp no)
-		(fields_autoplaced yes)
-		(property "Reference" "U1"
-			(at 97.3933 53.34 0)
-			(effects
-				(font
-					(size 1.27 1.27)
-				)
-				(justify left)
-			)
-		)
-		(property "Value" "4060"
-			(at 97.3933 55.88 0)
-			(effects
-				(font
-					(size 1.27 1.27)
-				)
-				(justify left)
-			)
-		)
-		(property "Footprint" ""
-			(at 95.25 76.2 0)
-			(effects
-				(font
-					(size 1.27 1.27)
-				)
-				(hide yes)
-			)
-		)
-		(property "Datasheet" "https://www.st.com/resource/en/datasheet/m74hc4060.pdf"
-			(at 95.25 78.74 0)
-			(effects
-				(font
-					(size 1.27 1.27)
-				)
-				(hide yes)
-			)
-		)
-		(property "Description" "Binary counter (14-stages) and oscillator"
-			(at 95.25 73.66 0)
-			(effects
-				(font
-					(size 1.27 1.27)
-				)
-				(hide yes)
-			)
-		)
-		(pin "1"
-		)
-		(pin "10"
-		)
-		(pin "7"
-		)
-		(pin "4"
-		)
-		(pin "9"
-		)
-		(pin "8"
-		)
-		(pin "14"
-		)
-		(pin "13"
-		)
-		(pin "11"
-		)
-		(pin "12"
-		)
-		(pin "3"
-		)
-		(pin "15"
-		)
-		(pin "16"
-		)
-		(pin "6"
-		)
-		(pin "5"
-		)
-		(pin "2"
-		)
-		(instances
-			(project ""
-				(path "/614b9759-e400-4d9a-b999-e6a52a22018a"
-					(reference "U1")
-					(unit 1)
-				)
-			)
-		)
-	)
 	(sheet_instances
 		(path "/"
