File: 2026-tractor.kicad_sch (KiCad schematic)
At the start: 0 parts

Commit message: Add updates
Parts:
- added BT1: Battery, symbol Device:Battery
- added CAN, Seat1: Conn_01x02, symbol Connector_Generic:Conn_01x02
- added F1: Pi Fuse (5A), symbol Device:Fuse
- added F2: System Fuse (20A), symbol Device:Fuse
- added J1: Conn_01x16, symbol Connector_Generic:Conn_01x16
- added J2: Interface Connector, symbol Connector_Generic:Conn_01x05
- added J3: Pi Pinout, symbol Connector_Generic:Conn_02x20_Odd_Even
- added J4: 12V-5V, symbol Connector_Generic:Conn_02x02_Counter_Clockwise
- added J5: Throttle Pedal, symbol Connector_Generic:Conn_01x03
- added J6: Pi USB, symbol Connector_Generic:Conn_01x02
- added NeutralSwitch, OperatorKill: SW_SPST, symbol Switch:SW_SPST
- added SW1: Kill Switch, symbol Switch:SW_SPST
- added SW2: Key Switch, symbol Switch:SW_Rotary_1x3_MP
Connections:
- new net: NeutralSwitch.1 (A), Seat1.2 (Pin_2)
- new net: NeutralSwitch.2 (B), SW2.3
- new net: F2.1, SW1.1 (A)
- new net: BT1.1 (+), F2.2
- new net 12V: F1.1, J4.1 (Pin_1)
- new net 5V: J4.4 (Pin_4), J6.1 (Pin_1)
- new net CAN CS: J3.24 (Pin_24)
- new net CAN H: CAN.1 (Pin_1), J1.15 (Pin_15), J2.4 (Pin_4)
- new net CAN INT: J3.22 (Pin_22)
- new net CAN L: CAN.2 (Pin_2), J1.2 (Pin_2), J2.5 (Pin_5)
- new net CAN MISO: J3.21 (Pin_21)
- new net CAN MOSI: J3.19 (Pin_19)
- new net CAN SCK: J3.23 (Pin_23)
- new net Engine MIL: J1.5 (Pin_5), J3.18 (Pin_18)
- new net Engine Oil: J1.4 (Pin_4), J3.16 (Pin_16)
- new net GND: BT1.2 (-), J2.2 (Pin_2), J4.2 (Pin_2), J4.3 (Pin_3), J6.2 (Pin_2)
- new net Ignition: J1.10 (Pin_10), SW2.2
- new net Kill Switch: J1.11 (Pin_11), J2.3 (Pin_3), OperatorKill.1 (A)
- new net Screen GND: J3.6 (Pin_6)
- new net Screen Power: J3.2 (Pin_2), J3.4 (Pin_4)
- new net Start: J1.7 (Pin_7), Seat1.1 (Pin_1)
- new net Throttle 5V: J1.12 (Pin_12), J5.3 (Pin_3)
- new net Throttle GND: J1.14 (Pin_14), J5.1 (Pin_1)
- new net Throttle SIG: J1.13 (Pin_13), J5.2 (Pin_2)
- new net VBAT (A): F1.2, J2.1 (Pin_1), OperatorKill.2 (B), SW1.2 (B), SW2.4, SW2.MP
Other:
- note added: "A"
- note added: "B"
- note added: "C"
- note added: "D"
- note added: "E"
- note added: "F"
- note added: "G"
- note added: "H"
- note added: "J"
- note added: "K"
- note added: "L"
- note added: "M"
- note added: "N"
- note added: "P"
- note added: "R"
- note added: "S"
