File: Tractor_Diagnostic.kicad_sch (KiCad schematic)
At the start: 3 parts

Commit message: second wiring option
Parts:
- added BT1: Battery_Cell, symbol Device:Battery_Cell
- added F2, F4: Fuse, symbol Device:Fuse
Connections:
- net GND: now also BT1.2 (-)
- new net: BT1.1 (+), F2.1, F4.1, F4.2
- no-connect marks 6 -> 15
